Commit message: optimal trajectory calculation for abb irb 6640 and abb irb 2600

File: model/irb6640.urdf (robot description, URDF)
Before this commit: robot abb_irb6640, 9 links, 8 joints
Links:
- added link link_cylinder, mass 210; collision mesh filename=/home/geekayman/based_on_flobaroid/model/meshes/irb6640_185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; visual mesh filename=/home/geekayman/based_on_flobaroid/model/meshes/irb6640_185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
- link support: mass 92.5052 -> 600
Joints:
- removed joint arm_to_world_fixed
- added joint box_support: type fixed, parent world, child support, origin xyz=0 0 0 rpy=0 0 0
- added joint joint_cylinder: type fixed, parent lwr_1_link, child link_cylinder, origin xyz=-0.365 -0.1895 0.405 rpy=0 -0.170 0
- joint base_joint_support: origin xyz=0 0 0.05 rpy=0 0 0 -> xyz=0 0 0 rpy=0 0 0
- joint lwr_0_joint: limit lower=-2.967 upper=2.967 effort=1000 velocity=1.7453 -> lower=-2.967 upper=2.967 effort=6700 velocity=1.7453; origin xyz=0 0 0.780 rpy=0 0 0 -> xyz=0 0 0.227 rpy=0 0 0
- joint lwr_1_joint: limit lower=-1.134 upper=1.4855 effort=1000 velocity=1.5707 -> lower=-1.134 upper=1.4855 effort=6300 velocity=1.5707; origin xyz=0.320 0 0 rpy=0 0 0 -> xyz=0.322 0.03 0.551 rpy=0 0 0
- joint lwr_2_joint: limit lower=-3.142 upper=1.222 effort=1000 velocity=1.5707 -> lower=-3.142 upper=1.222 effort=6500 velocity=1.5707
- joint lwr_3_joint: limit lower=-5.236 upper=5.236 effort=1000 velocity=2.9671 -> lower=-5.236 upper=5.236 effort=990 velocity=2.9671
- joint lwr_4_joint: limit lower=-2.094 upper=2.094 effort=1000 velocity=2.4435 -> lower=-2.094 upper=2.094 effort=1300 velocity=2.4435
- joint lwr_5_joint: limit lower=-6.283 upper=6.283 effort=1000 velocity=3.3161 -> lower=-6.283 upper=6.283 effort=500 velocity=3.3161; origin xyz=0.2 0 0 rpy=0 0 0 -> xyz=0.153 0 0 rpy=0 0 0
